Commit message: Add quadruped SLAM Nav2 competition autonomy

File: src/quadruped_description/urdf/quadruped.urdf.xacro (robot description, xacro)
@@ -1,12 +1,22 @@
 <?xml version="1.0"?>
-<robot xmlns:xacro="http://www.ros.org/wiki/xacro" name="quadruped">
+<robot xmlns:xacro="http://www.ros.org/wiki/xacro" name="wakula_quadruped">
+  <!-- Generic 12-DOF quadruped model for RViz and ros2_control debugging.
+       Replace these dimensions and inertias with measured hardware values before deployment. -->
   <xacro:property name="body_length" value="0.52"/>
   <xacro:property name="body_width" value="0.24"/>
   <xacro:property name="body_height" value="0.12"/>
+  <xacro:property name="hip_length" value="0.065"/>
   <xacro:property name="upper_leg_length" value="0.22"/>
   <xacro:property name="lower_leg_length" value="0.23"/>
   <xacro:property name="leg_radius" value="0.025"/>
-  <xacro:macro name="box_inertial" params="mass x y z">
+  <xacro:property name="foot_radius" value="0.035"/>
+  <material name="wakula_blue"><color rgba="0.06 0.28 0.62 1"/></material>
+  <material name="joint_gray"><color rgba="0.22 0.25 0.29 1"/></material>
+  <material name="leg_silver"><color rgba="0.68 0.72 0.76 1"/></material>
+  <material name="foot_black"><color rgba="0.04 0.04 0.04 1"/></material>
+  <material name="sensor_black"><color rgba="0.08 0.08 0.09 1"/></material>
+  <xacro:macro name="box_inertial" params="mass x y z ox:=0 oy:=0 oz:=0">
     <inertial>
+      <origin xyz="${ox} ${oy} ${oz}"/>
       <mass value="${mass}"/>
       <inertia ixx="${mass * (y*y + z*z) / 12.0}" ixy="0" ixz="0"
@@ -15,83 +25,160 @@
     </inertial>
   </xacro:macro>
+  <xacro:macro name="sphere_inertial" params="mass radius">
+    <inertial>
+      <mass value="${mass}"/>
+      <inertia ixx="${0.4 * mass * radius * radius}" ixy="0" ixz="0"
+               iyy="${0.4 * mass * radius * radius}" iyz="0"
+               izz="${0.4 * mass * radius * radius}"/>
+    </inertial>
+  </xacro:macro>
+  <!-- base_footprint remains on the nominal ground plane for navigation. -->
   <link name="base_footprint"/>
+  <joint name="base_footprint_joint" type="fixed">
+    <parent link="base_footprint"/>
+    <child link="base_link"/>
+    <origin xyz="0 0 0.44"/>
+  </joint>
   <link name="base_link">
     <visual>
       <geometry><box size="${body_length} ${body_width} ${body_height}"/></geometry>
-      <material name="body_blue"><color rgba="0.08 0.25 0.55 1"/></material>
+      <material name="wakula_blue"/>
     </visual>
-    <collision><geometry><box size="${body_length} ${body_width} ${body_height}"/></geometry></collision>
+    <collision>
+      <geometry><box size="${body_length} ${body_width} ${body_height}"/></geometry>
+    </collision>
     <xacro:box_inertial mass="12.0" x="${body_length}" y="${body_width}" z="${body_height}"/>
   </link>
-  <joint name="base_footprint_joint" type="fixed">
-    <parent link="base_footprint"/><child link="base_link"/>
-    <origin xyz="0 0 0.48"/>
-  </joint>
+  <!-- side is +1 for left legs and -1 for right legs. -->
   <xacro:macro name="leg" params="prefix x y side">
     <link name="${prefix}_hip_link">
-      <visual><geometry><cylinder radius="${leg_radius}" length="0.10"/></geometry></visual>
-      <collision><geometry><cylinder radius="${leg_radius}" length="0.10"/></geometry></collision>
-      <xacro:box_inertial mass="0.55" x="0.05" y="0.05" z="0.10"/>
+      <visual>
+        <origin xyz="0 ${side * hip_length / 2.0} 0" rpy="${pi/2} 0 0"/>
+        <geometry><cylinder radius="${leg_radius}" length="${hip_length}"/></geometry>
+        <material name="joint_gray"/>
+      </visual>
+      <collision>
+        <origin xyz="0 ${side * hip_length / 2.0} 0" rpy="${pi/2} 0 0"/>
+        <geometry><cylinder radius="${leg_radius}" length="${hip_length}"/></geometry>
+      </collision>
+      <xacro:box_inertial mass="0.55" x="${2*leg_radius}" y="${hip_length}"
+                           z="${2*leg_radius}" oy="${side * hip_length / 2.0}"/>
     </link>
     <joint name="${prefix}_hip_joint" type="revolute">
-      <parent link="base_link"/><child link="${prefix}_hip_link"/>
-      <origin xyz="${x} ${y} 0" rpy="${pi/2} 0 0"/>
-      <axis xyz="1 0 0"/><limit lower="-0.75" upper="0.75" effort="80" velocity="8"/>
+      <parent link="base_link"/>
+      <child link="${prefix}_hip_link"/>
+      <origin xyz="${x} ${y} 0"/>
+      <axis xyz="1 0 0"/>
+      <limit lower="-0.75" upper="0.75" effort="80" velocity="8"/>
+      <dynamics damping="0.2" friction="0.05"/>
     </joint>
     <link name="${prefix}_upper_leg">
-      <visual><origin xyz="0 0 ${-upper_leg_length/2}"/><geometry><cylinder radius="${leg_radius}" length="${upper_leg_length}"/></geometry></visual>
-      <collision><origin xyz="0 0 ${-upper_leg_length/2}"/><geometry><cylinder radius="${leg_radius}" length="${upper_leg_length}"/></geometry></collision>
-      <xacro:box_inertial mass="1.0" x="0.05" y="0.05" z="${upper_leg_length}"/>
+      <visual>
+        <origin xyz="0 0 ${-upper_leg_length/2.0}"/>
+        <geometry><cylinder radius="${leg_radius}" length="${upper_leg_length}"/></geometry>
+        <material name="leg_silver"/>
+      </visual>
+      <collision>
+        <origin xyz="0 0 ${-upper_leg_length/2.0}"/>
+        <geometry><cylinder radius="${leg_radius}" length="${upper_leg_length}"/></geometry>
+      </collision>
+      <xacro:box_inertial mass="1.0" x="${2*leg_radius}" y="${2*leg_radius}"
+                           z="${upper_leg_length}" oz="${-upper_leg_length/2.0}"/>
     </link>
     <joint name="${prefix}_thigh_joint" type="revolute">
-      <parent link="${prefix}_hip_link"/><child link="${prefix}_upper_leg"/>
-      <origin xyz="0 0 ${-0.05}"/>
-      <axis xyz="0 1 0"/><limit lower="-1.57" upper="1.20" effort="120" velocity="10"/>
+      <parent link="${prefix}_hip_link"/>
+      <child link="${prefix}_upper_leg"/>
+      <origin xyz="0 ${side * hip_length} 0"/>
+      <axis xyz="0 1 0"/>
+      <limit lower="-1.57" upper="1.20" effort="120" velocity="10"/>
+      <dynamics damping="0.25" friction="0.05"/>
     </joint>
     <link name="${prefix}_lower_leg">
-      <visual><origin xyz="0 0 ${-lower_leg_length/2}"/><geometry><cylinder radius="${leg_radius * 0.8}" length="${lower_leg_length}"/></geometry></visual>
-      <collision><origin xyz="0 0 ${-lower_leg_length/2}"/><geometry><cylinder radius="${leg_radius * 0.8}" length="${lower_leg_length}"/></geometry></collision>
-      <xacro:box_inertial mass="0.65" x="0.04" y="0.04" z="${lower_leg_length}"/>
+      <visual>
+        <origin xyz="0 0 ${-lower_leg_length/2.0}"/>
+        <geometry><cylinder radius="${leg_radius * 0.8}" length="${lower_leg_length}"/></geometry>
+        <material name="leg_silver"/>
+      </visual>
+      <collision>
+        <origin xyz="0 0 ${-lower_leg_length/2.0}"/>
+        <geometry><cylinder radius="${leg_radius * 0.8}" length="${lower_leg_length}"/></geometry>
+      </collision>
+      <xacro:box_inertial mass="0.65" x="${1.6*leg_radius}" y="${1.6*leg_radius}"
+                           z="${lower_leg_length}" oz="${-lower_leg_length/2.0}"/>
     </link>
     <joint name="${prefix}_calf_joint" type="revolute">
-      <parent link="${prefix}_upper_leg"/><child link="${prefix}_lower_leg"/>
+      <parent link="${prefix}_upper_leg"/>
+      <child link="${prefix}_lower_leg"/>
       <origin xyz="0 0 ${-upper_leg_length}"/>
-      <axis xyz="0 1 0"/><limit lower="-2.70" upper="-0.15" effort="120" velocity="10"/>
+      <axis xyz="0 1 0"/>
+      <limit lower="-2.70" upper="-0.15" effort="120" velocity="10"/>
+      <dynamics damping="0.25" friction="0.05"/>
     </joint>
     <link name="${prefix}_foot">
-      <visual><geometry><sphere radius="0.035"/></geometry></visual>
-      <collision><geometry><sphere radius="0.035"/></geometry></collision>
-      <xacro:box_inertial mass="0.12" x="0.07" y="0.07" z="0.07"/>
+      <visual>
+        <geometry><sphere radius="${foot_radius}"/></geometry>
+        <material name="foot_black"/>
+      </visual>
+      <collision><geometry><sphere radius="${foot_radius}"/></geometry></collision>
+      <xacro:sphere_inertial mass="0.12" radius="${foot_radius}"/>
     </link>
     <joint name="${prefix}_foot_joint" type="fixed">
-      <parent link="${prefix}_lower_leg"/><child link="${prefix}_foot"/>
+      <parent link="${prefix}_lower_leg"/>
+      <child link="${prefix}_foot"/>
       <origin xyz="0 0 ${-lower_leg_length}"/>
     </joint>
   </xacro:macro>
-  <xacro:leg prefix="front_left"  x="0.20"  y="0.15"  side="1"/>
-  <xacro:leg prefix="front_right" x="0.20"  y="-0.15" side="-1"/>
-  <xacro:leg prefix="rear_left"   x="-0.20" y="0.15"  side="1"/>
-  <xacro:leg prefix="rear_right"  x="-0.20" y="-0.15" side="-1"/>
+  <xacro:leg prefix="front_left"  x="0.20"  y="${body_width/2.0}"  side="1"/>
+  <xacro:leg prefix="front_right" x="0.20"  y="${-body_width/2.0}" side="-1"/>
+  <xacro:leg prefix="rear_left"   x="-0.20" y="${body_width/2.0}"  side="1"/>
+  <xacro:leg prefix="rear_right"  x="-0.20" y="${-body_width/2.0}" side="-1"/>
+  <!-- Sensor frames used by SLAM and terrain-perception nodes. -->
+  <link name="imu_link">
+    <visual><geometry><box size="0.04 0.03 0.015"/></geometry><material name="sensor_black"/></visual>
+    <xacro:box_inertial mass="0.03" x="0.04" y="0.03" z="0.015"/>
+  </link>
+  <joint name="imu_joint" type="fixed">
+    <parent link="base_link"/><child link="imu_link"/><origin xyz="0 0 0.065"/>
+  </joint>
+  <link name="lidar_link">
+    <visual><geometry><cylinder radius="0.045" length="0.04"/></geometry><material name="sensor_black"/></visual>
+    <xacro:box_inertial mass="0.18" x="0.09" y="0.09" z="0.04"/>
+  </link>
+  <joint name="lidar_joint" type="fixed">
+    <parent link="base_link"/><child link="lidar_link"/><origin xyz="0 0 0.085"/>
+  </joint>
+  <link name="camera_link">
+    <visual><geometry><box size="0.04 0.09 0.035"/></geometry><material name="sensor_black"/></visual>
+    <xacro:box_inertial mass="0.09" x="0.04" y="0.09" z="0.035"/>
+  </link>
+  <joint name="camera_joint" type="fixed">
+    <parent link="base_link"/><child link="camera_link"/><origin xyz="0.275 0 0.015"/>
+  </joint>
+  <link name="camera_optical_frame"/>
+  <joint name="camera_optical_joint" type="fixed">
+    <parent link="camera_link"/><child link="camera_optical_frame"/>
+    <origin rpy="${-pi/2} 0 ${-pi/2}"/>
+  </joint>
   <ros2_control name="QuadrupedSystem" type="system">
     <hardware><plugin>mock_components/GenericSystem</plugin></hardware>
-    <xacro:macro name="controlled_joint" params="name">
+    <xacro:macro name="controlled_joint" params="name initial:=0.0">
       <joint name="${name}">
         <command_interface name="position"/>
-        <state_interface name="position"><param name="initial_value">0.0</param></state_interface>
+        <state_interface name="position"><param name="initial_value">${initial}</param></state_interface>
         <state_interface name="velocity"/>
       </joint>
     </xacro:macro>
     <xacro:controlled_joint name="front_left_hip_joint"/>
-    <xacro:controlled_joint name="front_left_thigh_joint"/>
-    <xacro:controlled_joint name="front_left_calf_joint"/>
+    <xacro:controlled_joint name="front_left_thigh_joint" initial="0.55"/>
+    <xacro:controlled_joint name="front_left_calf_joint" initial="-1.10"/>
     <xacro:controlled_joint name="front_right_hip_joint"/>
-    <xacro:controlled_joint name="front_right_thigh_joint"/>
-    <xacro:controlled_joint name="front_right_calf_joint"/>
+    <xacro:controlled_joint name="front_right_thigh_joint" initial="0.55"/>
+    <xacro:controlled_joint name="front_right_calf_joint" initial="-1.10"/>
     <xacro:controlled_joint name="rear_left_hip_joint"/>
-    <xacro:controlled_joint name="rear_left_thigh_joint"/>
-    <xacro:controlled_joint name="rear_left_calf_joint"/>
+    <xacro:controlled_joint name="rear_left_thigh_joint" initial="0.55"/>
+    <xacro:controlled_joint name="rear_left_calf_joint" initial="-1.10"/>
     <xacro:controlled_joint name="rear_right_hip_joint"/>
-    <xacro:controlled_joint name="rear_right_thigh_joint"/>
-    <xacro:controlled_joint name="rear_right_calf_joint"/>
+    <xacro:controlled_joint name="rear_right_thigh_joint" initial="0.55"/>
+    <xacro:controlled_joint name="rear_right_calf_joint" initial="-1.10"/>
   </ros2_control>
 </robot>

Commit message: Document sensor selection and mounting

File: src/quadruped_description/urdf/quadruped.urdf.xacro (robot description, xacro)
@@ -146,5 +146,6 @@
   </link>
   <joint name="lidar_joint" type="fixed">
-    <parent link="base_link"/><child link="lidar_link"/><origin xyz="0 0 0.085"/>
+    <!-- Nominal top-center reservation; replace with measured scan-center TF. -->
+    <parent link="base_link"/><child link="lidar_link"/><origin xyz="0.04 0 0.12"/>
   </joint>
   <link name="camera_link">
@@ -153,5 +154,7 @@
   </link>
   <joint name="camera_joint" type="fixed">
-    <parent link="base_link"/><child link="camera_link"/><origin xyz="0.275 0 0.015"/>
+    <!-- Nominal front-center reservation with 12-degree downward pitch. -->
+    <parent link="base_link"/><child link="camera_link"/>
+    <origin xyz="0.29 0 0.03" rpy="0 ${12*pi/180} 0"/>
   </joint>
   <link name="camera_optical_frame"/>

Commit message: Add simulation and basic quadruped motion stack

File: src/quadruped_description/urdf/quadruped.urdf.xacro (robot description, xacro)
@@ -1,4 +1,7 @@
 <?xml version="1.0"?>
 <robot xmlns:xacro="http://www.ros.org/wiki/xacro" name="wakula_quadruped">
+  <!-- The same model targets GenericSystem, Gazebo or a future real plugin. -->
+  <xacro:arg name="simulation" default="false"/>
+  <xacro:arg name="controllers_file" default=""/>
   <!-- Generic 12-DOF quadruped model for RViz and ros2_control debugging.
        Replace these dimensions and inertias with measured hardware values before deployment. -->
@@ -128,4 +131,8 @@
       <origin xyz="0 0 ${-lower_leg_length}"/>
     </joint>
+    <gazebo reference="${prefix}_foot">
+      <mu1>1.5</mu1>
+      <mu2>1.5</mu2>
+    </gazebo>
   </xacro:macro>
   <xacro:leg prefix="front_left"  x="0.20"  y="${body_width/2.0}"  side="1"/>
@@ -158,5 +165,8 @@
     <origin xyz="0.29 0 0.03" rpy="0 ${12*pi/180} 0"/>
   </joint>
-  <link name="camera_optical_frame"/>
+  <link name="camera_optical_frame">
+    <!-- Tiny inertia keeps the preserved optical frame valid during URDF->SDF conversion. -->
+    <xacro:box_inertial mass="0.001" x="0.001" y="0.001" z="0.001"/>
+  </link>
   <joint name="camera_optical_joint" type="fixed">
     <parent link="camera_link"/><child link="camera_optical_frame"/>
@@ -164,5 +174,13 @@
   </joint>
   <ros2_control name="QuadrupedSystem" type="system">
-    <hardware><plugin>mock_components/GenericSystem</plugin></hardware>
+    <hardware>
+      <xacro:if value="$(arg simulation)">
+        <plugin>gz_ros2_control/GazeboSimSystem</plugin>
+      </xacro:if>
+      <xacro:unless value="$(arg simulation)">
+        <!-- Replace only this plugin when the selected real actuator SDK is known. -->
+        <plugin>mock_components/GenericSystem</plugin>
+      </xacro:unless>
+    </hardware>
     <xacro:macro name="controlled_joint" params="name initial:=0.0">
       <joint name="${name}">
@@ -185,3 +203,68 @@
     <xacro:controlled_joint name="rear_right_calf_joint" initial="-1.10"/>
   </ros2_control>
+  <!-- Gazebo-only physics, controller and sensor systems.  Real drivers keep
+       publishing the same ROS topics, so perception and navigation do not change. -->
+  <xacro:if value="$(arg simulation)">
+    <gazebo>
+      <self_collide>true</self_collide>
+      <plugin filename="gz_ros2_control-system"
+              name="gz_ros2_control::GazeboSimROS2ControlPlugin">
+        <parameters>$(arg controllers_file)</parameters>
+        <hold_joints>true</hold_joints>
+        <position_proportional_gain>0.25</position_proportional_gain>
+      </plugin>
+      <plugin filename="gz-sim-odometry-publisher-system"
+              name="gz::sim::systems::OdometryPublisher">
+        <odom_frame>odom</odom_frame>
+        <robot_base_frame>base_footprint</robot_base_frame>
+        <odom_topic>/odom</odom_topic>
+        <tf_topic>/tf</tf_topic>
+        <odom_publish_frequency>50</odom_publish_frequency>
+      </plugin>
+    </gazebo>
+    <gazebo reference="lidar_joint"><preserveFixedJoint>true</preserveFixedJoint></gazebo>
+    <gazebo reference="lidar_link">
+      <sensor name="wakula_lidar" type="gpu_lidar">
+        <always_on>true</always_on>
+        <update_rate>12</update_rate>
+        <visualize>false</visualize>
+        <topic>/scan</topic>
+        <lidar>
+          <scan><horizontal>
+            <samples>720</samples><resolution>1</resolution>
+            <min_angle>-${pi}</min_angle><max_angle>${pi}</max_angle>
+          </horizontal></scan>
+          <range><min>0.12</min><max>20.0</max><resolution>0.01</resolution></range>
+          <noise><type>gaussian</type><mean>0.0</mean><stddev>0.006</stddev></noise>
+        </lidar>
+      </sensor>
+    </gazebo>
+    <gazebo reference="camera_joint"><preserveFixedJoint>true</preserveFixedJoint></gazebo>
+    <gazebo reference="camera_optical_joint"><preserveFixedJoint>true</preserveFixedJoint></gazebo>
+    <gazebo reference="camera_link">
+      <sensor name="wakula_rgbd" type="rgbd_camera">
+        <always_on>true</always_on>
+        <update_rate>15</update_rate>
+        <visualize>false</visualize>
+        <topic>/rgbd_camera</topic>
+        <camera>
+          <horizontal_fov>1.40</horizontal_fov>
+          <image><width>640</width><height>360</height><format>R8G8B8</format></image>
+          <clip><near>0.20</near><far>8.0</far></clip>
+          <!-- Gazebo RGBD points use x-forward/y-left/z-up coordinates.  Label
+               them camera_link; real optical drivers continue using the fixed
+               camera_optical_frame supplied above. -->
+          <optical_frame_id>camera_link</optical_frame_id>
+          <noise><type>gaussian</type><mean>0.0</mean><stddev>0.002</stddev></noise>
+        </camera>
+      </sensor>
+    </gazebo>
+    <gazebo reference="imu_joint"><preserveFixedJoint>true</preserveFixedJoint></gazebo>
+    <gazebo reference="imu_link">
+      <sensor name="wakula_imu" type="imu">
+        <always_on>true</always_on><update_rate>100</update_rate>
+        <topic>/imu/data</topic>
+      </sensor>
+    </gazebo>
+  </xacro:if>
 </robot>
